File: kicad/BeanBoardSPI.kicad_sch (KiCad schematic)
At the start: 23 parts, among them J1 Beanboard Power, J10 SPI_6, J2 Beanboard Address, J3 Beanboard Data / Control, J4 SPI_0, J5 SPI_1, J6 SPI_2, J7 SPI_3, J8 SPI_4, J9 SPI_5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

Commit message: Update BeanBoardSPI.kicad_sch
Parts:
- added C1, C10, C2, C3, C4, C5, C6, C7, C8, C9: 0.1uF, Capacitor_THT:C_Disc_D5.0mm_W2.5mm_P2.50mm, symbol Device:C
- added J12: GPO, Connector_PinHeader_2.54mm:PinHeader_1x10_P2.54mm_Vertical, symbol Connector:Conn_01x10_Pin
- J1: value Beanboard Power -> Power; footprint (none) -> Connector_PinHeader_2.54mm:PinHeader_1x03_P2.54mm_Vertical
- J10, J4, J5, J6, J7, J8, J9: footprint (none) -> Connector_PinHeader_2.54mm:PinHeader_1x07_P2.54mm_Vertical; symbol Connector:Conn_01x06_Pin -> Connector:Conn_01x07_Pin
- J2: value Beanboard Address -> Address; footprint (none) -> Connector_PinHeader_2.54mm:PinHeader_1x16_P2.54mm_Vertical
- J3: value Beanboard Data / Control -> Data / Control; footprint (none) -> Connector_PinHeader_2.54mm:PinHeader_1x16_P2.54mm_Vertical
- JP1: value Jumper_2_Open -> CLK; footprint (none) -> Connector_PinHeader_2.54mm:PinHeader_1x02_P2.54mm_Vertical
- JP2: value Jumper_2_Open -> CLK/2; footprint (none) -> Connector_PinHeader_2.54mm:PinHeader_1x02_P2.54mm_Vertical
- JP3: value Jumper_2_Bridged -> CLK/4; footprint (none) -> Connector_PinHeader_2.54mm:PinHeader_1x02_P2.54mm_Vertical
- U1, U3: footprint (none) -> Package_DIP:DIP-16_W7.62mm_Socket
- U2, U4: footprint (none) -> Package_DIP:DIP-20_W7.62mm_Socket
- U5, U6, U7, U8, U9: footprint (none) -> Package_DIP:DIP-14_W7.62mm_Socket
Connections:
- net GND: now also J10.3 (Pin_3), J4.3 (Pin_3), J5.3 (Pin_3), J6.3 (Pin_3), J7.3 (Pin_3), J8.3 (Pin_3), J9.3 (Pin_3); no longer J10.6 (Pin_6), J4.6 (Pin_6), J5.6 (Pin_6), J6.6 (Pin_6), J7.6 (Pin_6), J8.6 (Pin_6), J9.6 (Pin_6)
- net SCLK: now also J10.4 (Pin_4), J4.4 (Pin_4), J5.4 (Pin_4), J6.4 (Pin_4), J7.4 (Pin_4), J8.4 (Pin_4), J9.4 (Pin_4); no longer J10.2 (Pin_2), J4.2 (Pin_2), J5.2 (Pin_2), J6.2 (Pin_2), J7.2 (Pin_2), J8.2 (Pin_2), J9.2 (Pin_2)
- net SER_OUT: now also J10.6 (Pin_6), J4.6 (Pin_6), J5.6 (Pin_6), J6.6 (Pin_6), J7.6 (Pin_6), J8.6 (Pin_6), J9.6 (Pin_6); no longer J10.4 (Pin_4), J4.4 (Pin_4), J5.4 (Pin_4), J6.4 (Pin_4), J7.4 (Pin_4), J8.4 (Pin_4), J9.4 (Pin_4)
- net ~{CS_0}: now also J4.7 (Pin_7); no longer J4.3 (Pin_3)
- net ~{CS_1}: now also J5.7 (Pin_7); no longer J5.3 (Pin_3)
- net ~{CS_2}: now also J6.7 (Pin_7); no longer J6.3 (Pin_3)
- net ~{CS_3}: now also J7.7 (Pin_7); no longer J7.3 (Pin_3)
- net ~{CS_4}: now also J8.7 (Pin_7); no longer J8.3 (Pin_3)
- net ~{CS_5}: now also J9.7 (Pin_7); no longer J9.3 (Pin_3)
- net ~{CS_6}: now also J10.7 (Pin_7); no longer J10.3 (Pin_3)
- no-connect marks 34 -> 51
Other:
- note added: "Beanboard Connectors"
- note added: "GPO connector for physical stability only"
- moved on the sheet: U1, U10, U2, U3, U4, U5A, U5B, U5C, U5D, U5E, U6A, U6B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

Commit message: Update BeanBoardSPI.kicad_sch
Parts:
- J10: value SPI_6 -> SPI6
- J4: value SPI_0 -> SPI0 (RA8875); footprint Connector_PinHeader_2.54mm:PinHeader_1x07_P2.54mm_Vertical -> Connector_PinHeader_2.54mm:PinHeader_1x15_P2.54mm_Vertical; symbol Connector:Conn_01x07_Pin -> Connector:Conn_01x15_Pin
- J5: value SPI_1 -> SPI1
- J6: value SPI_2 -> SPI2
- J7: value SPI_3 -> SPI3
- J8: value SPI_4 -> SPI4
- J9: value SPI_5 -> SPI5
Connections:
- net +5V: now also C1.1, C10.1, C2.1, C3.1, C4.1, C5.1, C6.1, C7.1, C8.1, C9.1
- net GND: now also C1.2, C10.2, C2.2, C3.2, C4.2, C5.2, C6.2, C7.2, C8.2, C9.2, J4.2 (Pin_2); no longer J4.3 (Pin_3)
- net SCLK: now also J4.5 (Pin_5); no longer J4.4 (Pin_4)
- net SER_IN: now also J4.6 (Pin_6); no longer J4.5 (Pin_5)
- net SER_OUT: now also J4.7 (Pin_7); no longer J4.6 (Pin_6)
- net ~{CS_0}: now also J4.8 (Pin_8); no longer J4.7 (Pin_7)
- net ~{SRESET}: now also J4.9 (Pin_9)
- no-connect marks 51 -> 58

Commit message: Update BeanBoardSPI.kicad_sch
Parts:
- added J11: GPO, Connector_PinSocket_2.54mm:PinSocket_1x10_P2.54mm_Vertical, symbol Connector:Conn_01x10_Socket
- added J13: GPI, Connector_PinHeader_2.54mm:PinHeader_1x10_P2.54mm_Vertical, symbol Connector:Conn_01x10_Pin
- added J14: GPI, Connector_PinSocket_2.54mm:PinSocket_1x10_P2.54mm_Vertical, symbol Connector:Conn_01x10_Socket
Connections:
- net at J12.1 (Pin_1): now also J11.1 (Pin_1)
- net at J12.10 (Pin_10): now also J11.10 (Pin_10)
- net at J12.2 (Pin_2): now also J11.2 (Pin_2)
- net at J12.3 (Pin_3): now also J11.3 (Pin_3)
- net at J12.4 (Pin_4): now also J11.4 (Pin_4)
- net at J12.5 (Pin_5): now also J11.5 (Pin_5)
- net at J12.6 (Pin_6): now also J11.6 (Pin_6)
- net at J12.7 (Pin_7): now also J11.7 (Pin_7)
- net at J12.8 (Pin_8): now also J11.8 (Pin_8)
- net at J12.9 (Pin_9): now also J11.9 (Pin_9)
- new net: J13.1 (Pin_1), J14.1 (Pin_1)
- new net: J13.10 (Pin_10), J14.10 (Pin_10)
- new net: J13.2 (Pin_2), J14.2 (Pin_2)
- new net: J13.3 (Pin_3), J14.3 (Pin_3)
- new net: J13.4 (Pin_4), J14.4 (Pin_4)
- new net: J13.5 (Pin_5), J14.5 (Pin_5)
- new net: J13.6 (Pin_6), J14.6 (Pin_6)
- new net: J13.7 (Pin_7), J14.7 (Pin_7)
- new net: J13.8 (Pin_8), J14.8 (Pin_8)
- new net: J13.9 (Pin_9), J14.9 (Pin_9)
- no-connect marks 58 -> 48
Other:
- note removed: "GPO connector for physical stability only"
Changed lines of the file:
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@@
   (no_connect (at 60.96 24.13))
   (no_connect (at 157.48 134.62))
-  (no_connect (at 78.74 27.94))
   (no_connect (at 78.74 19.05))
   (no_connect (at 224.79 30.48))
-  (no_connect (at 78.74 35.56))
   (no_connect (at 110.49 87.63))
   (no_connect (at 39.37 24.13))
-  (no_connect (at 78.74 45.72))
   (no_connect (at 224.79 22.86))
-  (no_connect (at 78.74 48.26))
-  (no_connect (at 78.74 38.1))
   (no_connect (at 39.37 31.75))
   (no_connect (at 224.79 35.56))
@@
   (no_connect (at 224.79 25.4))
   (no_connect (at 157.48 132.08))
-  (no_connect (at 78.74 33.02))
   (no_connect (at 39.37 44.45))
-  (no_connect (at 78.74 30.48))
   (no_connect (at 157.48 162.56))
-  (no_connect (at 78.74 50.8))
   (no_connect (at 39.37 49.53))
   (no_connect (at 157.48 160.02))
@@
   (no_connect (at 195.58 129.54))
   (no_connect (at 224.79 38.1))
-  (no_connect (at 78.74 40.64))
   (no_connect (at 157.48 152.4))
-  (no_connect (at 78.74 43.18))
   (no_connect (at 39.37 29.21))
   (no_connect (at 39.37 41.91))
@@
     (effects (font (size 1.27 1.27)) (justify left bottom))
   )
-  (text "GPO connector \nfor physical \nstability \nonly" (at 83.82 50.8 0)
-    (effects (font (size 1.27 1.27)) (justify left bottom))
-  )
   (text "USB\nKeyboard\nLCD\nGPIO" (at 111.76 80.01 0)
     (effects (font (size 1.27 1.27)) (justify left bottom))
@@
     )
   )
+  (symbol (lib_id "Connector:Conn_01x10_Socket") (at 99.06 38.1 0) (unit 1)
+    (in_bom yes) (on_board yes) (dnp no)
+    (property "Reference" "J14" (at 99.06 53.34 0)
+      (effects (font (size 1.27 1.27)))
+    )
+    (property "Value" "GPI" (at 99.06 24.13 0)
+      (effects (font (size 1.27 1.27)))
+    )
+    (property "Footprint" "Connector_PinSocket_2.54mm:PinSocket_1x10_P2.54mm_Vertical" (at 99.06 38.1 0)
+      (effects (font (size 1.27 1.27)) hide)
+    )
+    (property "Datasheet" "~" (at 99.06 38.1 0)
+      (effects (font (size 1.27 1.27)) hide)
+    )
+    (pin "5")
+    (pin "4")
+    (pin "6")
+    (pin "3")
+    (pin "7")
+    (pin "1")
+    (pin "10")
+    (pin "2")
+    (pin "8")
+    (pin "9")
+    (instances
+      (project "BeanBoardSPI"
+        (path "/6c08ad2a-e233-4d4c-8add-9bc0e49a4487"
+          (reference "J14") (unit 1)
+        )
+      )
+    )
+  )
   (symbol (lib_id "74xx:74LS00") (at 124.46 130.81 0) (unit 5)
     (in_bom yes) (on_board yes) (dnp no) (fields_autoplaced)
@@
   (symbol (lib_id "Connector:Conn_01x10_Pin") (at 73.66 38.1 0) (unit 1)
     (in_bom yes) (on_board yes) (dnp no)
-    (property "Reference" "J12" (at 80.01 24.13 0)
+    (property "Reference" "J12" (at 73.66 53.34 0)
       (effects (font (size 1.27 1.27)))
     )
@@
     )
   )
+  (symbol (lib_id "Connector:Conn_01x10_Pin") (at 88.9 38.1 0) (unit 1)
+    (in_bom yes) (on_board yes) (dnp no)
+    (property "Reference" "J13" (at 88.9 53.34 0)
+      (effects (font (size 1.27 1.27)))
+    )
+    (property "Value" "GPI" (at 90.17 24.13 0)
+      (effects (font (size 1.27 1.27)))
+    )
+    (property "Footprint" "Connector_PinHeader_2.54mm:PinHeader_1x10_P2.54mm_Vertical" (at 88.9 38.1 0)
+      (effects (font (size 1.27 1.27)) hide)
+    )
+    (property "Datasheet" "~" (at 88.9 38.1 0)
+      (effects (font (size 1.27 1.27)) hide)
+    )
+    (pin "5")
+    (pin "4")
+    (pin "6")
+    (pin "3")
+    (pin "7")
+    (pin "1")
+    (pin "10")
+    (pin "2")
+    (pin "8")
+    (pin "9")
+    (instances
+      (project "BeanBoardSPI"
+        (path "/6c08ad2a-e233-4d4c-8add-9bc0e49a4487"
+          (reference "J13") (unit 1)
+        )
+      )
+    )
+  )
   (symbol (lib_id "Connector:Conn_01x16_Pin") (at 34.29 31.75 0) (unit 1)
     (in_bom yes) (on_board yes) (dnp no)
@@
         )
       )
+    )
+  )
+  (symbol (lib_id "Connector:Conn_01x10_Socket") (at 83.82 38.1 0) (unit 1)
+    (in_bom yes) (on_board yes) (dnp no)
+    (property "Reference" "J11" (at 83.82 53.34 0)
+      (effects (font (size 1.27 1.27)))
+    )
+    (property "Value" "GPO" (at 83.82 24.13 0)
+      (effects (font (size 1.27 1.27)))
+    )
+    (property "Footprint" "Connector_PinSocket_2.54mm:PinSocket_1x10_P2.54mm_Vertical" (at 83.82 38.1 0)
+      (effects (font (size 1.27 1.27)) hide)
+    )
+    (property "Datasheet" "~" (at 83.82 38.1 0)
+      (effects (font (size 1.27 1.27)) hide)
+    )
+    (pin "5")
+    (pin "4")
+    (pin "6")
+    (pin "3")
+    (pin "7")
+    (pin "1")
+    (pin "10")
+    (pin "2")
+    (pin "8")
+    (pin "9")
+    (instances
+      (project "BeanBoardSPI"
+        (path "/6c08ad2a-e233-4d4c-8add-9bc0e49a4487"
+          (reference "J11") (unit 1)
+        )
+      )

Commit message: Update BeanBoardSPI.kicad_sch
Parts:
- added J15: Power, Connector_PinSocket_2.54mm:PinSocket_1x03_P2.54mm_Vertical, symbol Connector:Conn_01x03_Socket
Connections:
- net +5V: now also J15.2 (Pin_2)
- net GND: now also J1.3 (Pin_3), J15.1 (Pin_1), J15.3 (Pin_3)
- no-connect marks 48 -> 47
Other:
- moved on the sheet: J1
Changed lines of the file:
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@@
   (junction (at 6.35 78.74) (diameter 0) (color 0 0 0 0)
   )
+  (junction (at 85.09 11.43) (diameter 0) (color 0 0 0 0)
+  )
   (junction (at 226.06 73.66) (diameter 0) (color 0 0 0 0)
   )
-  (junction (at 82.55 13.97) (diameter 0) (color 0 0 0 0)
-  )
   (junction (at 233.68 102.87) (diameter 0) (color 0 0 0 0)
   )
@@
   (junction (at 6.35 116.84) (diameter 0) (color 0 0 0 0)
   )
+  (junction (at 95.25 11.43) (diameter 0) (color 0 0 0 0)
+  )
+  (junction (at 85.09 13.97) (diameter 0) (color 0 0 0 0)
+  )
   (junction (at 6.35 40.64) (diameter 0) (color 0 0 0 0)
   )
+  (junction (at 80.01 11.43) (diameter 0) (color 0 0 0 0)
+  )
   (junction (at 6.35 15.24) (diameter 0) (color 0 0 0 0)
   )
@@
   )
   (junction (at 13.97 116.84) (diameter 0) (color 0 0 0 0)
-  )
-  (junction (at 82.55 16.51) (diameter 0) (color 0 0 0 0)
   )
   (no_connect (at 60.96 19.05))
@@
   (no_connect (at 60.96 24.13))
   (no_connect (at 157.48 134.62))
-  (no_connect (at 78.74 19.05))
   (no_connect (at 224.79 30.48))
   (no_connect (at 110.49 87.63))
@@
     (stroke (width 0) (type default))
   )
+  (wire (pts (xy 80.01 11.43) (xy 78.74 11.43))
+    (stroke (width 0) (type default))
+  )
+  (wire (pts (xy 96.52 16.51) (xy 95.25 16.51))
+    (stroke (width 0) (type default))
+  )
   (wire (pts (xy 46.99 76.2) (xy 46.99 83.82))
     (stroke (width 0) (type default))
@@
     (stroke (width 0) (type default))
   )
-  (wire (pts (xy 90.17 16.51) (xy 82.55 16.51))
+  (wire (pts (xy 78.74 13.97) (xy 85.09 13.97))
     (stroke (width 0) (type default))
   )
@@
     (stroke (width 0) (type default))
   )
-  (wire (pts (xy 82.55 13.97) (xy 78.74 13.97))
+  (wire (pts (xy 80.01 11.43) (xy 85.09 11.43))
     (stroke (width 0) (type default))
   )
@@
     (stroke (width 0) (type default))
   )
+  (wire (pts (xy 85.09 11.43) (xy 95.25 11.43))
+    (stroke (width 0) (type default))
+  )
   (wire (pts (xy 210.82 97.79) (xy 210.82 100.33))
     (stroke (width 0) (type default))
@@
     (stroke (width 0) (type default))
   )
-  (wire (pts (xy 90.17 13.97) (xy 82.55 13.97))
-    (stroke (width 0) (type default))
-  )
   (wire (pts (xy 210.82 66.04) (xy 226.06 66.04))
     (stroke (width 0) (type default))
@@
     (stroke (width 0) (type default))
   )
+  (wire (pts (xy 80.01 11.43) (xy 80.01 16.51))
+    (stroke (width 0) (type default))
+  )
   (wire (pts (xy 110.49 85.09) (xy 124.46 85.09))
     (stroke (width 0) (type default))
@@
     (stroke (width 0) (type default))
   )
+  (wire (pts (xy 95.25 11.43) (xy 96.52 11.43))
+    (stroke (width 0) (type default))
+  )
   (wire (pts (xy 233.68 102.87) (xy 246.38 102.87))
     (stroke (width 0) (type default))
@@
     (stroke (width 0) (type default))
   )
+  (wire (pts (xy 85.09 13.97) (xy 96.52 13.97))
+    (stroke (width 0) (type default))
+  )
   (wire (pts (xy 54.61 92.71) (xy 46.99 92.71))
     (stroke (width 0) (type default))
@@
     (stroke (width 0) (type default))
   )
-  (wire (pts (xy 82.55 16.51) (xy 78.74 16.51))
-    (stroke (width 0) (type default))
-  )
   (wire (pts (xy 124.46 102.87) (xy 124.46 91.44))
     (stroke (width 0) (type default))
   )
+  (wire (pts (xy 78.74 16.51) (xy 80.01 16.51))
+    (stroke (width 0) (type default))
+  )
   (wire (pts (xy 233.68 110.49) (xy 233.68 102.87))
     (stroke (width 0) (type default))
@@
     (stroke (width 0) (type default))
   )
+  (wire (pts (xy 95.25 11.43) (xy 95.25 16.51))
+    (stroke (width 0) (type default))
+  )
   (wire (pts (xy 226.06 60.96) (xy 227.33 60.96))
     (stroke (width 0) (type default))
@@
     (effects (font (size 1.27 1.27)) (justify right bottom))
   )
-  (label "GND" (at 90.17 13.97 0) (fields_autoplaced)
+  (label "GND" (at 90.17 11.43 0) (fields_autoplaced)
     (effects (font (size 1.27 1.27)) (justify left bottom))
   )
@@
     (effects (font (size 1.27 1.27)) (justify left bottom))
   )
-  (label "+5V" (at 90.17 16.51 0) (fields_autoplaced)
+  (label "+5V" (at 90.17 13.97 0) (fields_autoplaced)
     (effects (font (size 1.27 1.27)) (justify left bottom))
   )
@@
     )
   )
-  (symbol (lib_id "Connector:Conn_01x03_Pin") (at 73.66 16.51 0) (unit 1)
-    (in_bom yes) (on_board yes) (dnp no)
-    (property "Reference" "J1" (at 74.295 6.35 0)
-      (effects (font (size 1.27 1.27)))
-    )
-    (property "Value" "Power" (at 76.2 8.89 0)
-      (effects (font (size 1.27 1.27)))
-    )
-    (property "Footprint" "Connector_PinHeader_2.54mm:PinHeader_1x03_P2.54mm_Vertical" (at 73.66 16.51 0)
-      (effects (font (size 1.27 1.27)) hide)
-    )
-    (property "Datasheet" "~" (at 73.66 16.51 0)
+  (symbol (lib_id "Connector:Conn_01x03_Pin") (at 73.66 13.97 0) (unit 1)
+    (in_bom yes) (on_board yes) (dnp no)
+    (property "Reference" "J1" (at 74.295 3.81 0)
+      (effects (font (size 1.27 1.27)))
+    )
+    (property "Value" "Power" (at 76.2 6.35 0)
+      (effects (font (size 1.27 1.27)))
+    )
+    (property "Footprint" "Connector_PinHeader_2.54mm:PinHeader_1x03_P2.54mm_Vertical" (at 73.66 13.97 0)
+      (effects (font (size 1.27 1.27)) hide)
+    )
+    (property "Datasheet" "~" (at 73.66 13.97 0)
       (effects (font (size 1.27 1.27)) hide)
     )
@@
     )
   )
+  (symbol (lib_id "Connector:Conn_01x03_Socket") (at 101.6 13.97 0) (unit 1)
+    (in_bom yes) (on_board yes) (dnp no)
+    (property "Reference" "J15" (at 102.235 3.81 0)
+      (effects (font (size 1.27 1.27)))
+    )
+    (property "Value" "Power" (at 104.14 6.35 0)
+      (effects (font (size 1.27 1.27)))
+    )
+    (property "Footprint" "Connector_PinSocket_2.54mm:PinSocket_1x03_P2.54mm_Vertical" (at 101.6 13.97 0)
+      (effects (font (size 1.27 1.27)) hide)
+    )
+    (property "Datasheet" "~" (at 101.6 13.97 0)
+      (effects (font (size 1.27 1.27)) hide)
+    )
+    (pin "1")
+    (pin "3")
+    (pin "2")
+    (instances
+      (project "BeanBoardSPI"
+        (path "/6c08ad2a-e233-4d4c-8add-9bc0e49a4487"
+          (reference "J15") (unit 1)
+        )
+      )
+    )
+  )
   (symbol (lib_id "74xx:74LS00") (at 254 113.03 0) (unit 1)
     (in_bom yes) (on_board yes) (dnp no)
@@
     )
   )
-  (symbol (lib_id "power:PWR_FLAG") (at 82.55 16.51 0) (mirror x) (unit 1)
-    (in_bom yes) (on_board yes) (dnp no)
-    (property "Reference" "#FLG02" (at 82.55 18.415 0)
-      (effects (font (size 1.27 1.27)) hide)
-    )
-    (property "Value" "PWR_FLAG" (at 85.09 19.05 0)
-      (effects (font (size 1.27 1.27)))
-    )
-    (property "Footprint" "" (at 82.55 16.51 0)
-      (effects (font (size 1.27 1.27)) hide)
-    )
-    (property "Datasheet" "~" (at 82.55 16.51 0)
+  (symbol (lib_id "power:PWR_FLAG") (at 85.09 13.97 0) (mirror x) (unit 1)
+    (in_bom yes) (on_board yes) (dnp no)
+    (property "Reference" "#FLG02" (at 85.09 15.875 0)
+      (effects (font (size 1.27 1.27)) hide)
+    )
+    (property "Value" "PWR_FLAG" (at 87.63 17.78 0)
+      (effects (font (size 1.27 1.27)))
+    )
+    (property "Footprint" "" (at 85.09 13.97 0)
+      (effects (font (size 1.27 1.27)) hide)
+    )
+    (property "Datasheet" "~" (at 85.09 13.97 0)
       (effects (font (size 1.27 1.27)) hide)
     )
@@
     )
   )
-  (symbol (lib_id "power:PWR_FLAG") (at 82.55 13.97 0) (unit 1)
-    (in_bom yes) (on_board yes) (dnp no)
-    (property "Reference" "#FLG01" (at 82.55 12.065 0)
-      (effects (font (size 1.27 1.27)) hide)
-    )
-    (property "Value" "PWR_FLAG" (at 85.09 11.43 0)
-      (effects (font (size 1.27 1.27)))
-    )
-    (property "Footprint" "" (at 82.55 13.97 0)
-      (effects (font (size 1.27 1.27)) hide)
-    )
-    (property "Datasheet" "~" (at 82.55 13.97 0)
-      (effects (font (size 1.27 1.27)) hide)
-    )
+  (symbol (lib_id "power:PWR_FLAG") (at 85.09 11.43 0) (unit 1)
+    (in_bom yes) (on_board yes) (dnp no)
+    (property "Reference" "#FLG01" (at 85.09 9.525 0)
+      (effects (font (size 1.27 1.27)) hide)
+    )
+    (property "Value" "PWR_FLAG" (at 87.63 7.62 0)
+      (effects (font (size 1.27 1.27)))
+    )
+    (property "Footprint" "" (at 85.09 11.43 0)
+      (effects (font (size 1.27 1.27)) hide)
+    )
+    (property "Datasheet" "~" (at 85.09 11.43 0)
+      (effects (font (size 1.27 1.27)) hide)
+    )
