File: kicad/BeanBoardSPI.kicad_pcb (KiCad board)
At the start: 4 copper layers, 0 parts

Commit message: Update BeanBoardSPI.kicad_pcb
Parts:
- added C1: 0.1uF, Capacitor_THT:C_Disc_D5.0mm_W2.5mm_P2.50mm, F.Cu at (155.3, -36.1)
- added C10: 0.1uF, Capacitor_THT:C_Disc_D5.0mm_W2.5mm_P2.50mm, F.Cu at (161.8, -24.0)
- added C2: 0.1uF, Capacitor_THT:C_Disc_D5.0mm_W2.5mm_P2.50mm, F.Cu at (155.3, -32.1)
- added C3: 0.1uF, Capacitor_THT:C_Disc_D5.0mm_W2.5mm_P2.50mm, F.Cu at (155.3, -28.0)
- added C4: 0.1uF, Capacitor_THT:C_Disc_D5.0mm_W2.5mm_P2.50mm, F.Cu at (155.3, -24.0)
- added C5: 0.1uF, Capacitor_THT:C_Disc_D5.0mm_W2.5mm_P2.50mm, F.Cu at (155.3, -19.9)
- added C6: 0.1uF, Capacitor_THT:C_Disc_D5.0mm_W2.5mm_P2.50mm, F.Cu at (155.3, -15.9)
- added C7: 0.1uF, Capacitor_THT:C_Disc_D5.0mm_W2.5mm_P2.50mm, F.Cu at (161.8, -36.1)
- added C8: 0.1uF, Capacitor_THT:C_Disc_D5.0mm_W2.5mm_P2.50mm, F.Cu at (161.8, -32.1)
- added C9: 0.1uF, Capacitor_THT:C_Disc_D5.0mm_W2.5mm_P2.50mm, F.Cu at (161.8, -28.0)
- added J1: Power, Connector_PinHeader_2.54mm:PinHeader_1x03_P2.54mm_Vertical, F.Cu at (288.8, 20.0)
- added J10: SPI_6, Connector_PinHeader_2.54mm:PinHeader_1x07_P2.54mm_Vertical, F.Cu at (138.9, -40.9)
- added J12: GPO, Connector_PinHeader_2.54mm:PinHeader_1x10_P2.54mm_Vertical, F.Cu at (289.8, 55.8)
- added J2: Address, Connector_PinHeader_2.54mm:PinHeader_1x16_P2.54mm_Vertical, F.Cu at (144.0, 20.1)
- added J3: Data / Control, Connector_PinHeader_2.54mm:PinHeader_1x16_P2.54mm_Vertical, F.Cu at (154.0, 20.0)
- added J4: SPI_0, Connector_PinHeader_2.54mm:PinHeader_1x07_P2.54mm_Vertical, F.Cu at (111.0, -40.9)
- added J5: SPI_1, Connector_PinHeader_2.54mm:PinHeader_1x07_P2.54mm_Vertical, F.Cu at (115.7, -40.9)
- added J6: SPI_2, Connector_PinHeader_2.54mm:PinHeader_1x07_P2.54mm_Vertical, F.Cu at (120.3, -40.9)
- added J7: SPI_3, Connector_PinHeader_2.54mm:PinHeader_1x07_P2.54mm_Vertical, F.Cu at (125.0, -40.9)
- added J8: SPI_4, Connector_PinHeader_2.54mm:PinHeader_1x07_P2.54mm_Vertical, F.Cu at (129.6, -40.9)
- added J9: SPI_5, Connector_PinHeader_2.54mm:PinHeader_1x07_P2.54mm_Vertical, F.Cu at (134.3, -40.9)
- added JP1: CLK, Connector_PinHeader_2.54mm:PinHeader_1x02_P2.54mm_Vertical, F.Cu at (111.0, -6.10)
- added JP2: CLK/2, Connector_PinHeader_2.54mm:PinHeader_1x02_P2.54mm_Vertical, F.Cu at (111.0, -10.9)
- added JP3: CLK/4, Connector_PinHeader_2.54mm:PinHeader_1x02_P2.54mm_Vertical, F.Cu at (111.3, -16.3)
- added U1: 74LS42, Package_DIP:DIP-16_W7.62mm_Socket, F.Cu at (110.8, -63.1)
- added U10: 74LS138, Package_DIP:DIP-16_W7.62mm_Socket, F.Cu at (134.3, -63.1)
- added U2: 74LS299, Package_DIP:DIP-20_W7.62mm_Socket, F.Cu at (155.3, -63.1)
- added U3: 74LS161, Package_DIP:DIP-16_W7.62mm_Socket, F.Cu at (122.5, -63.1)
- added U4: 74LS373, Package_DIP:DIP-20_W7.62mm_Socket, F.Cu at (167.1, -63.1)
- added U5: 74LS00, Package_DIP:DIP-14_W7.62mm_Socket, F.Cu at (110.8, -82.6)
- added U6: 74LS00, Package_DIP:DIP-14_W7.62mm_Socket, F.Cu at (122.5, -82.6)
- added U7: 74LS04, Package_DIP:DIP-14_W7.62mm_Socket, F.Cu at (134.3, -82.6)
- added U8: 74LS02, Package_DIP:DIP-14_W7.62mm_Socket, F.Cu at (146.0, -82.6)
- added U9: 74LS74, Package_DIP:DIP-14_W7.62mm_Socket, F.Cu at (157.8, -82.6)

Commit message: Update BeanBoardSPI.kicad_pcb
Parts:
- J10: value SPI_6 -> SPI6
- J4: value SPI_0 -> SPI0 (RA8875); footprint Connector_PinHeader_2.54mm:PinHeader_1x07_P2.54mm_Vertical -> Connector_PinHeader_2.54mm:PinHeader_1x15_P2.54mm_Vertical
- J5: value SPI_1 -> SPI1
- J6: value SPI_2 -> SPI2
- J7: value SPI_3 -> SPI3
- J8: value SPI_4 -> SPI4
- J9: value SPI_5 -> SPI5
- moved C1 133.2 mm to (286.4, -12.7)
- moved C10 133.2 mm to (292.9, -0.52)
- moved C2 133.2 mm to (286.4, -8.62)
- moved C3 133.2 mm to (286.4, -4.57)
- moved C4 133.2 mm to (286.4, -0.52)
- moved C5 133.2 mm to (286.4, 3.53)
- moved C6 133.2 mm to (286.4, 7.58)
- moved C7 133.2 mm to (292.9, -12.7)
- moved C8 133.2 mm to (292.9, -8.62)
- moved C9 133.2 mm to (292.9, -4.57)
- moved J4 94.7 mm to (110.7, 53.8), turned to 90 degrees
- moved JP1 2.55 mm to (111.3, -8.64)
- moved JP2 1.54 mm to (111.3, -12.4)
Connections:
- C1 pad 1: unconnected-(C1-Pad1) -> /+5V
- C1 pad 2: unconnected-(C1-Pad2) -> /GND
- C10 pad 1: unconnected-(C10-Pad1) -> /+5V
- C10 pad 2: unconnected-(C10-Pad2) -> /GND
- C2 pad 1: unconnected-(C2-Pad1) -> /+5V
- C2 pad 2: unconnected-(C2-Pad2) -> /GND
- C3 pad 1: unconnected-(C3-Pad1) -> /+5V
- C3 pad 2: unconnected-(C3-Pad2) -> /GND
- C4 pad 1: unconnected-(C4-Pad1) -> /+5V
- C4 pad 2: unconnected-(C4-Pad2) -> /GND
- C5 pad 1: unconnected-(C5-Pad1) -> /+5V
- C5 pad 2: unconnected-(C5-Pad2) -> /GND
- C6 pad 1: unconnected-(C6-Pad1) -> /+5V
- C6 pad 2: unconnected-(C6-Pad2) -> /GND
- C7 pad 1: unconnected-(C7-Pad1) -> /+5V
- C7 pad 2: unconnected-(C7-Pad2) -> /GND
- C8 pad 1: unconnected-(C8-Pad1) -> /+5V
- C8 pad 2: unconnected-(C8-Pad2) -> /GND
- C9 pad 1: unconnected-(C9-Pad1) -> /+5V
- C9 pad 2: unconnected-(C9-Pad2) -> /GND
- J4 pad 2: unconnected-(J4-Pin_2-Pad2) -> /GND
- J4 pad 3: /GND -> unconnected-(J4-Pin_3-Pad3)
- J4 pad 4: /SCLK -> unconnected-(J4-Pin_4-Pad4)
- J4 pad 5: /SER_IN -> /SCLK
- J4 pad 6: /SER_OUT -> /SER_IN
- J4 pad 7: /~{CS_0} -> /SER_OUT
Other:
- board outline added: 199.4 x 80 mm

Commit message: Update BeanBoardSPI.kicad_pcb
Parts:
- moved J10 178.0 mm to (269.1, 80.5), turned to 90 degrees
- moved J9 159.7 mm to (238.1, 80.5), turned to 90 degrees
- moved J8 144.0 mm to (207.0, 80.5), turned to 90 degrees
- moved J7 131.7 mm to (176.0, 80.5), turned to 90 degrees
- moved J6 123.9 mm to (144.9, 80.5), turned to 90 degrees
- moved J5 121.4 mm to (113.9, 80.5), turned to 90 degrees
- moved JP2 31.7 mm to (140.0, 0.73)
- moved JP3 31.7 mm to (140.0, -3.09)
- moved JP1 31.7 mm to (140.0, 4.54)

Commit message: Update BeanBoardSPI.kicad_pcb
Parts:
- added J11: GPO, Connector_PinSocket_2.54mm:PinSocket_1x10_P2.54mm_Vertical, F.Cu at (296.7, 55.8)
- added J13: GPI, Connector_PinHeader_2.54mm:PinHeader_1x10_P2.54mm_Vertical, F.Cu at (287.3, 55.8)
- added J14: GPI, Connector_PinSocket_2.54mm:PinSocket_1x10_P2.54mm_Vertical, F.Cu at (293.4, 55.8)
- moved J10 9.77 mm to (259.3, 80.5)
- moved J9 7.82 mm to (230.2, 80.5)
- moved J8 5.86 mm to (201.1, 80.5)
- moved J7 3.91 mm to (172.1, 80.5)
- moved J6 1.95 mm to (143.0, 80.5)
Connections:
- J12 pad 1: unconnected-(J12-Pin_1-Pad1) -> Net-(J11-Pin_1)
- J12 pad 10: unconnected-(J12-Pin_10-Pad10) -> Net-(J11-Pin_10)
- J12 pad 2: unconnected-(J12-Pin_2-Pad2) -> Net-(J11-Pin_2)
- J12 pad 3: unconnected-(J12-Pin_3-Pad3) -> Net-(J11-Pin_3)
- J12 pad 4: unconnected-(J12-Pin_4-Pad4) -> Net-(J11-Pin_4)
- J12 pad 5: unconnected-(J12-Pin_5-Pad5) -> Net-(J11-Pin_5)
- J12 pad 6: unconnected-(J12-Pin_6-Pad6) -> Net-(J11-Pin_6)
- J12 pad 7: unconnected-(J12-Pin_7-Pad7) -> Net-(J11-Pin_7)
- J12 pad 8: unconnected-(J12-Pin_8-Pad8) -> Net-(J11-Pin_8)
- J12 pad 9: unconnected-(J12-Pin_9-Pad9) -> Net-(J11-Pin_9)

Commit message: Update BeanBoardSPI.kicad_pcb
Parts:
- added J15: Power, Connector_PinHeader_2.54mm:PinHeader_1x03_P2.54mm_Vertical, F.Cu at (288.8, 23.6)
Connections:
- J1 pad 3: unconnected-(J1-Pin_3-Pad3) -> /GND
Other:
- board text added: "GND"
- board text added: "VCC"

Commit message: Update BeanBoardSPI.kicad_pcb
Parts:
- J15: footprint Connector_PinHeader_2.54mm:PinHeader_1x03_P2.54mm_Vertical -> Connector_PinSocket_2.54mm:PinSocket_1x03_P2.54mm_Vertical
Changed lines of the file:
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@@
     )
   )
-  (footprint "Connector_PinHeader_2.54mm:PinHeader_1x03_P2.54mm_Vertical" (layer "F.Cu")
+  (footprint "Connector_PinSocket_2.54mm:PinSocket_1x03_P2.54mm_Vertical" (layer "F.Cu")
     (at 288.798745 23.552314 90)
-    (descr "Through hole straight pin header, 1x03, 2.54mm pitch, single row")
-    (tags "Through hole pin header THT 1x03 2.54mm single row")
+    (descr "Through hole straight socket strip, 1x03, 2.54mm pitch, single row (from Kicad 4.0.7), script generated")
+    (tags "Through hole socket strip THT 1x03 2.54mm single row")
     (property "Sheetfile" "BeanBoardSPI.kicad_sch")
     (property "Sheetname" "")
@@
     (property "ki_keywords" "connector")
     (attr through_hole)
-    (fp_text reference "J15" (at 0 -2.33 90) (layer "F.SilkS")
+    (fp_text reference "J15" (at 0 -2.77 90) (layer "F.SilkS")
         (effects (font (size 1 1) (thickness 0.15)))
     )
-    (fp_text value "Power" (at 0 7.41 90) (layer "F.Fab")
+    (fp_text value "Power" (at 0 7.85 90) (layer "F.Fab")
         (effects (font (size 1 1) (thickness 0.15)))
     )
-    (fp_text user "${REFERENCE}" (at 0 2.54) (layer "F.Fab")
+    (fp_text user "${REFERENCE}" (at 0 2.54 180) (layer "F.Fab")
         (effects (font (size 1 1) (thickness 0.15)))
     )
-    (fp_line (start -1.33 -1.33) (end 0 -1.33)
-      (stroke (width 0.12) (type solid)) (layer "F.SilkS"))
-    (fp_line (start -1.33 0) (end -1.33 -1.33)
-      (stroke (width 0.12) (type solid)) (layer "F.SilkS"))
     (fp_line (start -1.33 1.27) (end -1.33 6.41)
       (stroke (width 0.12) (type solid)) (layer "F.SilkS"))
@@
     (fp_line (start -1.33 6.41) (end 1.33 6.41)
       (stroke (width 0.12) (type solid)) (layer "F.SilkS"))
+    (fp_line (start 0 -1.33) (end 1.33 -1.33)
+      (stroke (width 0.12) (type solid)) (layer "F.SilkS"))
+    (fp_line (start 1.33 -1.33) (end 1.33 0)
+      (stroke (width 0.12) (type solid)) (layer "F.SilkS"))
     (fp_line (start 1.33 1.27) (end 1.33 6.41)
       (stroke (width 0.12) (type solid)) (layer "F.SilkS"))
-    (fp_line (start -1.8 -1.8) (end -1.8 6.85)
+    (fp_line (start -1.8 -1.8) (end 1.75 -1.8)
       (stroke (width 0.05) (type solid)) (layer "F.CrtYd"))
-    (fp_line (start -1.8 6.85) (end 1.8 6.85)
+    (fp_line (start -1.8 6.85) (end -1.8 -1.8)
       (stroke (width 0.05) (type solid)) (layer "F.CrtYd"))
-    (fp_line (start 1.8 -1.8) (end -1.8 -1.8)
+    (fp_line (start 1.75 -1.8) (end 1.75 6.85)
       (stroke (width 0.05) (type solid)) (layer "F.CrtYd"))
-    (fp_line (start 1.8 6.85) (end 1.8 -1.8)
+    (fp_line (start 1.75 6.85) (end -1.8 6.85)
       (stroke (width 0.05) (type solid)) (layer "F.CrtYd"))
-    (fp_line (start -1.27 -0.635) (end -0.635 -1.27)
+    (fp_line (start -1.27 -1.27) (end 0.635 -1.27)
       (stroke (width 0.1) (type solid)) (layer "F.Fab"))
-    (fp_line (start -1.27 6.35) (end -1.27 -0.635)
+    (fp_line (start -1.27 6.35) (end -1.27 -1.27)
       (stroke (width 0.1) (type solid)) (layer "F.Fab"))
-    (fp_line (start -0.635 -1.27) (end 1.27 -1.27)
+    (fp_line (start 0.635 -1.27) (end 1.27 -0.635)
       (stroke (width 0.1) (type solid)) (layer "F.Fab"))
-    (fp_line (start 1.27 -1.27) (end 1.27 6.35)
+    (fp_line (start 1.27 -0.635) (end 1.27 6.35)
       (stroke (width 0.1) (type solid)) (layer "F.Fab"))
     (fp_line (start 1.27 6.35) (end -1.27 6.35)
@@
     (pad "3" thru_hole oval (at 0 5.08 90) (size 1.7 1.7) (drill 1) (layers "*.Cu" "*.Mask")
       (net 1 "/GND") (pinfunction "Pin_3") (pintype "passive"))
-    (model "${KICAD6_3DMODEL_DIR}/Connector_PinHeader_2.54mm.3dshapes/PinHeader_1x03_P2.54mm_Vertical.wrl"
+    (model "${KICAD6_3DMODEL_DIR}/Connector_PinSocket_2.54mm.3dshapes/PinSocket_1x03_P2.54mm_Vertical.wrl"
       (offset (xyz 0 0 0))
       (scale (xyz 1 1 1))

Commit message: Update BeanBoardSPI.kicad_pcb
Parts:
- moved U5 202.5 mm to (268.2, 44.6)
- moved U3 166.6 mm to (250.7, 43.4)
- moved U6 164.5 mm to (250.7, 20.5)
- moved U1 162.2 mm to (233.1, 43.4)
- moved JP1 155.2 mm to (290.3, 43.4)
- moved JP2 155.2 mm to (290.3, 39.6)
- moved JP3 155.2 mm to (290.3, 35.7)
- moved U9 151.1 mm to (268.2, 20.5)
- moved U7 142.8 mm to (233.1, 20.5)
- moved U8 122.8 mm to (180.4, 35.2)
- moved U4 106.3 mm to (215.5, 31.4)
- moved U2 103.7 mm to (198.0, 31.4)
- moved U10 101.2 mm to (162.8, 34.0)
- moved J10 2.22 mm to (259.3, 82.7)
- moved J5 2.22 mm to (113.9, 82.7)
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Other:
- board text added: "PainfulDiodes"
Changed lines of the file:
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@@
   )
   (footprint "Connector_PinHeader_2.54mm:PinHeader_1x02_P2.54mm_Vertical" (layer "F.Cu")
-    (at 140.044 0.727 90)
+    (at 290.322745 39.554314 90)
     (descr "Through hole straight pin header, 1x02, 2.54mm pitch, single row")
     (tags "Through hole pin header THT 1x02 2.54mm single row")
@@
   )
   (footprint "Connector_PinHeader_2.54mm:PinHeader_1x07_P2.54mm_Vertical" (layer "F.Cu")
-    (at 142.968504 80.518 90)
+    (at 142.968504 82.734314 90)
     (descr "Through hole straight pin header, 1x07, 2.54mm pitch, single row")
     (tags "Through hole pin header THT 1x07 2.54mm single row")
@@
   )
   (footprint "Package_DIP:DIP-16_W7.62mm_Socket" (layer "F.Cu")
-    (at 110.756 -63.114)
+    (at 233.088077 43.359314)
     (descr "16-lead though-hole mounted DIP package, row spacing 7.62 mm (300 mils), Socket")
     (tags "THT DIP DIL PDIP 2.54mm 7.62mm 300mil Socket")
@@
   )
   (footprint "Package_DIP:DIP-14_W7.62mm_Socket" (layer "F.Cu")
-    (at 146.006 -82.614)
+    (at 180.383078 35.241314)
     (descr "14-lead though-hole mounted DIP package, row spacing 7.62 mm (300 mils), Socket")
     (tags "THT DIP DIL PDIP 2.54mm 7.62mm 300mil Socket")
@@
   )
   (footprint "Connector_PinHeader_2.54mm:PinHeader_1x07_P2.54mm_Vertical" (layer "F.Cu")
-    (at 230.239434 80.518 90)
+    (at 230.239434 82.734314 90)
     (descr "Through hole straight pin header, 1x07, 2.54mm pitch, single row")
     (tags "Through hole pin header THT 1x07 2.54mm single row")
@@
   )
   (footprint "Package_DIP:DIP-20_W7.62mm_Socket" (layer "F.Cu")
-    (at 167.056 -63.114)
+    (at 215.519744 31.441314)
     (descr "20-lead though-hole mounted DIP package, row spacing 7.62 mm (300 mils), Socket")
     (tags "THT DIP DIL PDIP 2.54mm 7.62mm 300mil Socket")
@@
   )
   (footprint "Package_DIP:DIP-14_W7.62mm_Socket" (layer "F.Cu")
-    (at 110.756 -82.614)
+    (at 268.224745 44.634314)
     (descr "14-lead though-hole mounted DIP package, row spacing 7.62 mm (300 mils), Socket")
     (tags "THT DIP DIL PDIP 2.54mm 7.62mm 300mil Socket")
@@
   )
   (footprint "Connector_PinHeader_2.54mm:PinHeader_1x07_P2.54mm_Vertical" (layer "F.Cu")
-    (at 172.058814 80.518 90)
+    (at 172.058814 82.734314 90)
     (descr "Through hole straight pin header, 1x07, 2.54mm pitch, single row")
     (tags "Through hole pin header THT 1x07 2.54mm single row")
@@
   )
   (footprint "Package_DIP:DIP-14_W7.62mm_Socket" (layer "F.Cu")
-    (at 157.756 -82.614)
+    (at 268.224745 20.504314)
     (descr "14-lead though-hole mounted DIP package, row spacing 7.62 mm (300 mils), Socket")
     (tags "THT DIP DIL PDIP 2.54mm 7.62mm 300mil Socket")
@@
   )
   (footprint "Connector_PinHeader_2.54mm:PinHeader_1x07_P2.54mm_Vertical" (layer "F.Cu")
-    (at 259.329745 80.518 90)
+    (at 259.329745 82.734314 90)
     (descr "Through hole straight pin header, 1x07, 2.54mm pitch, single row")
     (tags "Through hole pin header THT 1x07 2.54mm single row")
@@
   )
   (footprint "Package_DIP:DIP-20_W7.62mm_Socket" (layer "F.Cu")
-    (at 155.306 -63.114)
+    (at 197.951411 31.441314)
     (descr "20-lead though-hole mounted DIP package, row spacing 7.62 mm (300 mils), Socket")
     (tags "THT DIP DIL PDIP 2.54mm 7.62mm 300mil Socket")
@@
   )
   (footprint "Package_DIP:DIP-16_W7.62mm_Socket" (layer "F.Cu")
-    (at 122.506 -63.114)
+    (at 250.65641 43.359314)
     (descr "16-lead though-hole mounted DIP package, row spacing 7.62 mm (300 mils), Socket")
     (tags "THT DIP DIL PDIP 2.54mm 7.62mm 300mil Socket")
@@
   )
   (footprint "Connector_PinHeader_2.54mm:PinHeader_1x07_P2.54mm_Vertical" (layer "F.Cu")
-    (at 201.149124 80.518 90)
+    (at 201.149124 82.734314 90)
     (descr "Through hole straight pin header, 1x07, 2.54mm pitch, single row")
     (tags "Through hole pin header THT 1x07 2.54mm single row")
@@
   )
   (footprint "Connector_PinHeader_2.54mm:PinHeader_1x02_P2.54mm_Vertical" (layer "F.Cu")
-    (at 140.049 4.537 90)
+    (at 290.327745 43.364314 90)
     (descr "Through hole straight pin header, 1x02, 2.54mm pitch, single row")
     (tags "Through hole pin header THT 1x02 2.54mm single row")
@@
   )
   (footprint "Package_DIP:DIP-14_W7.62mm_Socket" (layer "F.Cu")
-    (at 134.256 -82.614)
+    (at 233.088077 20.504314)
     (descr "14-lead though-hole mounted DIP package, row spacing 7.62 mm (300 mils), Socket")
     (tags "THT DIP DIL PDIP 2.54mm 7.62mm 300mil Socket")
@@
   )
   (footprint "Connector_PinHeader_2.54mm:PinHeader_1x02_P2.54mm_Vertical" (layer "F.Cu")
-    (at 140.044 -3.088 90)
+    (at 290.322745 35.739314 90)
     (descr "Through hole straight pin header, 1x02, 2.54mm pitch, single row")
     (tags "Through hole pin header THT 1x02 2.54mm single row")
@@
   )
   (footprint "Package_DIP:DIP-14_W7.62mm_Socket" (layer "F.Cu")
-    (at 122.506 -82.614)
+    (at 250.65641 20.504314)
     (descr "14-lead though-hole mounted DIP package, row spacing 7.62 mm (300 mils), Socket")
     (tags "THT DIP DIL PDIP 2.54mm 7.62mm 300mil Socket")
@@
   )
   (footprint "Connector_PinHeader_2.54mm:PinHeader_1x07_P2.54mm_Vertical" (layer "F.Cu")
-    (at 113.878194 80.518 90)
+    (at 113.878194 82.734314 90)
     (descr "Through hole straight pin header, 1x07, 2.54mm pitch, single row")
     (tags "Through hole pin header THT 1x07 2.54mm single row")
@@
   )
   (footprint "Package_DIP:DIP-16_W7.62mm_Socket" (layer "F.Cu")
-    (at 134.256 -63.114)
+    (at 162.814745 33.966314)
     (descr "16-lead though-hole mounted DIP package, row spacing 7.62 mm (300 mils), Socket")
     (tags "THT DIP DIL PDIP 2.54mm 7.62mm 300mil Socket")
@@
   (gr_rect locked (start 101.6 14.732) (end 300.99 94.742)
     (stroke (width 0.1) (type default)) (fill none) (layer "Edge.Cuts"))
-  (gr_rect (start 227.841328 64.77) (end 247.907328 82.804)
+  (gr_rect (start 227.841328 66.986314) (end 247.907328 85.020314)
     (stroke (width 0.1) (type default)) (fill none) (layer "F.Fab"))
-  (gr_rect (start 140.589832 64.77) (end 160.655832 82.804)
+  (gr_rect (start 140.589832 66.986314) (end 160.655832 85.020314)
     (stroke (width 0.1) (type default)) (fill none) (layer "F.Fab"))
   (gr_rect locked (start 104.902 15.494) (end 152.908 55.626)
     (stroke (width 0.1) (type default)) (fill none) (layer "F.Fab"))
-  (gr_rect (start 111.506 64.77) (end 131.572 82.804)
+  (gr_rect (start 111.506 66.986314) (end 131.572 85.020314)
     (stroke (width 0.1) (type default)) (fill none) (layer "F.Fab"))
-  (gr_rect (start 198.757496 64.77) (end 218.823496 82.804)
+  (gr_rect (start 198.757496 66.986314) (end 218.823496 85.020314)
     (stroke (width 0.1) (type default)) (fill none) (layer "F.Fab"))
-  (gr_rect (start 256.925158 64.77) (end 276.991158 82.804)
+  (gr_rect (start 256.925158 66.986314) (end 276.991158 85.020314)
     (stroke (width 0.1) (type default)) (fill none) (layer "F.Fab"))
-  (gr_rect (start 169.673664 64.77) (end 189.739664 82.804)
+  (gr_rect (start 169.673664 66.986314) (end 189.739664 85.020314)
     (stroke (width 0.1) (type default)) (fill none) (layer "F.Fab"))
   (gr_circle locked (center 202.967859 24.870231) (end 203.475114 25.193917)
@@
     (effects (font (size 1 1) (thickness 0.15)) (justify left bottom))
   )
+  (gr_text "PainfulDiodes" (at 263.652745 91.878314) (layer "F.SilkS")
+    (effects (font (size 3 3) (thickness 0.375)) (justify left bottom))
+  )
   (gr_text locked "VIN\n\nGND\n\n3Vo\n\nLITE\n\nSCK\n\nMISO\n\nMOSI\n\nCS\n\nRST\n\nWAIT\n\nINT\n\nY+\n\nY-\n\nX-\n\nX+" (at 146.812 58.928 90) (layer "F.SilkS")
     (effects (font (size 0.79 0.79) (thickness 0.15)) (justify left bottom))
@@
     (effects (font (size 1 1) (thickness 0.15)) (justify left bottom))
   )
-  (gr_text locked "PainfulDiodes\nBeanBoard" (at 213.868 91.948) (layer "User.1")
-    (effects (font (size 3 3) (thickness 0.375)) (justify left bottom))
+  (gr_text locked "PainfulDiodes\nBeanBoard" (at 278.638745 171.126314) (layer "User.1")
+    (effects (font (size 1.5 1.5) (thickness 0.18)) (justify left bottom))
   )
   (gr_text locked "HD44780 LCD" (at 132.664175 41.991951) (layer "User.1")

Commit message: Update BeanBoardSPI.kicad_pcb
Parts:
- moved C7 132.3 mm to (167.9, 30.7)
- moved C1 110.1 mm to (185.7, 31.9)
- moved C2 90.9 mm to (203.2, 28.1)
- moved C8 81.0 mm to (220.7, 28.1)
- moved C9 70.6 mm to (238.3, 40.1)
- moved C10 55.0 mm to (255.8, 40.1)
- moved C3 52.8 mm to (238.3, 17.2)
- moved C4 43.8 mm to (273.3, 41.3)
- moved C5 33.5 mm to (255.8, 17.2)
- moved C6 16.2 mm to (273.3, 17.2)
- moved J14 9.65 mm to (283.7, 55.8)
- moved J11 3.33 mm to (293.4, 55.8)
Routing:
- added copper zone on In2.Cu, net /+5V
- added copper zone on In1.Cu, net /GND
Other:
- board text added: "GPI0"
- board text added: "GPI1"
- board text added: "GPI2"
- board text added: "GPI3"
- board text added: "GPI4"
- board text added: "GPI5"
- board text added: "GPI6"
- board text added: "GPI7"
- board text added: "GPO0"
- board text added: "GPO1"
- board text added: "GPO2"
- board text added: "GPO3"
- board text added: "GPO4"
- board text added: "GPO5"
- board text added: "GPO6"
- board text added: "GPO7"
- board text added: "~{GPIO_RD}"
- board text added: "~{RD}"
- board text added: "~{WR}"
