File: kicad/BeanBoardSPI.kicad_pcb (KiCad board)
At the start: 4 copper layers, 199.4 x 80 mm, 38 parts, among them J1 Power, J10 SPI6, J11 GPO, J12 GPO, J13 GPI, J14 GPI, J15 Power, J2 Address, J3 Data / Control, J4 SPI0 (RA8875)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

Commit message: Update BeanBoardSPI.kicad_pcb
Other:
- board text added: "SPI1"
- board text added: "SPI2"
- board text added: "SPI3"
- board text added: "SPI4"
- board text added: "SPI5"
- board text added: "SPI6"
Changed lines of the file:
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@@
         (effects (font (size 1 1) (thickness 0.15)))
     )
-    (fp_text value "74LS42" (at 3.81 20.11) (layer "F.Fab")
+    (fp_text value "74LS42" (at 3.81 20.11) (layer "F.SilkS")
         (effects (font (size 1 1) (thickness 0.15)))
     )
@@
         (effects (font (size 1 1) (thickness 0.15)))
     )
-    (fp_text value "74LS02" (at 3.81 17.57) (layer "F.Fab")
+    (fp_text value "74LS02" (at 3.81 17.57) (layer "F.SilkS")
         (effects (font (size 1 1) (thickness 0.15)))
     )
@@
         (effects (font (size 1 1) (thickness 0.15)))
     )
-    (fp_text value "74LS373" (at 3.81 25.19) (layer "F.Fab")
+    (fp_text value "74LS373" (at 3.81 25.19) (layer "F.SilkS")
         (effects (font (size 1 1) (thickness 0.15)))
     )
@@
         (effects (font (size 1 1) (thickness 0.15)))
     )
-    (fp_text value "74LS00" (at 3.81 17.57) (layer "F.Fab")
+    (fp_text value "74LS00" (at 3.81 17.57) (layer "F.SilkS")
         (effects (font (size 1 1) (thickness 0.15)))
     )
@@
         (effects (font (size 1 1) (thickness 0.15)))
     )
-    (fp_text value "74LS74" (at 3.81 17.57) (layer "F.Fab")
+    (fp_text value "74LS74" (at 3.81 17.57) (layer "F.SilkS")
         (effects (font (size 1 1) (thickness 0.15)))
     )
@@
         (effects (font (size 1 1) (thickness 0.15)))
     )
-    (fp_text value "74LS299" (at 3.81 25.19) (layer "F.Fab")
+    (fp_text value "74LS299" (at 3.81 25.19) (layer "F.SilkS")
         (effects (font (size 1 1) (thickness 0.15)))
     )
@@
         (effects (font (size 1 1) (thickness 0.15)))
     )
-    (fp_text value "74LS161" (at 3.81 20.11) (layer "F.Fab")
+    (fp_text value "74LS161" (at 3.81 20.11) (layer "F.SilkS")
         (effects (font (size 1 1) (thickness 0.15)))
     )
@@
         (effects (font (size 1 1) (thickness 0.15)))
     )
-    (fp_text value "74LS04" (at 3.81 17.57) (layer "F.Fab")
+    (fp_text value "74LS04" (at 3.81 17.57) (layer "F.SilkS")
         (effects (font (size 1 1) (thickness 0.15)))
     )
@@
         (effects (font (size 1 1) (thickness 0.15)))
     )
-    (fp_text value "74LS00" (at 3.81 17.57) (layer "F.Fab")
+    (fp_text value "74LS00" (at 3.81 17.57) (layer "F.SilkS")
         (effects (font (size 1 1) (thickness 0.15)))
     )
@@
         (effects (font (size 1 1) (thickness 0.15)))
     )
-    (fp_text value "74LS138" (at 3.81 20.11) (layer "F.Fab")
+    (fp_text value "74LS138" (at 3.81 20.11) (layer "F.SilkS")
         (effects (font (size 1 1) (thickness 0.15)))
     )
@@
     (effects (font (size 1 1) (thickness 0.15)) (justify left bottom))
   )
+  (gr_text "SPI5" (at 236.576345 78.924314) (layer "F.SilkS")
+    (effects (font (size 1 1) (thickness 0.15)) (justify left bottom))
+  )
   (gr_text "GPI0" (at 278.130745 56.533481) (layer "F.SilkS")
     (effects (font (size 1 1) (thickness 0.15)) (justify left bottom))
@@
     (effects (font (size 3 3) (thickness 0.375)) (justify left bottom))
   )
+  (gr_text "SPI1" (at 120.549145 78.924314) (layer "F.SilkS")
+    (effects (font (size 1 1) (thickness 0.15)) (justify left bottom))
+  )
   (gr_text "GPO6" (at 295.402745 71.653548) (layer "F.SilkS")
     (effects (font (size 1 1) (thickness 0.15)) (justify left bottom))
@@
     (effects (font (size 1 1) (thickness 0.15)) (justify left bottom))
   )
+  (gr_text "SPI2" (at 149.555945 78.924314) (layer "F.SilkS")
+    (effects (font (size 1 1) (thickness 0.15)) (justify left bottom))
+  )
   (gr_text "GPI3" (at 278.130745 64.08587) (layer "F.SilkS")
     (effects (font (size 1 1) (thickness 0.15)) (justify left bottom))
@@
     (effects (font (size 1 1) (thickness 0.15)) (justify left bottom))
   )
+  (gr_text "SPI4" (at 207.569545 78.924314) (layer "F.SilkS")
+    (effects (font (size 1 1) (thickness 0.15)) (justify left bottom))
+  )
   (gr_text "GND" (at 278.511697 79.432314) (layer "F.SilkS")
     (effects (font (size 1 1) (thickness 0.15)) (justify left bottom))
@@
     (effects (font (size 1 1) (thickness 0.15)) (justify left bottom))
   )
+  (gr_text "SPI3" (at 178.562745 78.924314) (layer "F.SilkS")
+    (effects (font (size 1 1) (thickness 0.15)) (justify left bottom))
+  )
   (gr_text "GPO7" (at 295.402745 74.167087) (layer "F.SilkS")
     (effects (font (size 1 1) (thickness 0.15)) (justify left bottom))
@@
     (effects (font (size 1 1) (thickness 0.15)) (justify left bottom))
   )
+  (gr_text "SPI6" (at 265.583145 78.924314) (layer "F.SilkS")
+    (effects (font (size 1 1) (thickness 0.15)) (justify left bottom))
+  )
   (gr_text locked "~{CLKINH}" (at 170.312102 27.799844 90) (layer "User.1")
     (effects (font (size 1 1) (thickness 0.15)) (justify left bottom))
@@
   (group "" locked (id 6be17e69-0b09-48e3-9b92-57c6ba02f2c8)
     (members
+      3a79ffd1-c576-4194-97c4-6083a72789c5
       8ccde5d4-0694-40fa-bb82-c2c9163c8cb5
+      90983100-eadc-4323-9460-d25cdcf20338
       dd73d9dc-a68e-4e19-8214-7ce93c573189
     )

Commit message: Update BeanBoardSPI.kicad_pcb
Routing:
- net /SCLK: track 0.00 -> 219.8 mm, vias 0 -> 6
- net /SER_IN: track 0.00 -> 207.0 mm, vias 0 -> 6
- net /SER_OUT: track 0.00 -> 194.4 mm, vias 0 -> 6
- net /~{CS_6}: track 0.00 -> 99.5 mm, vias 0 -> 2
- net /~{CS_2}: track 0.00 -> 87.4 mm, vias 0 -> 2
- net /~{CS_3}: track 0.00 -> 72.1 mm, vias 0 -> 2
- net /D4: track 0.00 -> 64.7 mm, vias 0 -> 3
- net /~{CS_5}: track 0.00 -> 62.7 mm, vias 0 -> 2
- net /~{WR}: track 0.00 -> 61.4 mm, vias 0 -> 1
- net /D5: track 0.00 -> 56.4 mm, vias 0 -> 1
- net /~{RD}: track 0.00 -> 51.7 mm, vias 0 -> 1
- net /D6: track 0.00 -> 51.3 mm, vias 0 -> 1
- net /A3: track 0.00 -> 45.8 mm, vias 0 -> 1
- net /~{CS_4}: track 0.00 -> 42.4 mm
- net /A2: track 0.00 -> 40.2 mm, vias 0 -> 1
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
Commit message: Update BeanBoardSPI.kicad_pcb
Routing:
- net /D3: track 11.0 -> 66.6 mm, vias 0 -> 3
- net /D1: track 19.2 -> 73.2 mm, vias 2 -> 4
- net /D2: track 18.6 -> 65.3 mm, vias 0 -> 2
- net /D0: track 29.1 -> 72.3 mm, vias 2 -> 4
- net /D7: track 21.0 -> 56.0 mm, vias 1 -> 2
- net /D4: track 64.7 -> 71.9 mm, vias 3 -> 5
- net /D5: track 56.4 -> 63.1 mm, vias 1 -> 3
- net /D6: track 51.3 -> 54.5 mm, vias 1 -> 3
- net /~{CS_4}: track 42.4 -> 43.7 mm, vias 0 -> 1
- net /~{CS_5}: track 62.7 -> 63.4 mm, vias 2 -> 3
- net /~{CS_6}: track 99.5 -> 100.2 mm, vias 2 -> 3

Commit message: Update BeanBoardSPI.kicad_pcb
Routing:
- net /INT_CLK: track 0.00 -> 159.3 mm, vias 0 -> 5
- net /CLK: track 0.00 -> 153.9 mm, vias 0 -> 2
- net /~{SRESET}: track 36.6 -> 178.9 mm, vias 2 -> 6
- net /~{CS_1}: track 0.00 -> 126.8 mm, vias 0 -> 2
- net /~{CS_0}: track 0.00 -> 123.3 mm, vias 0 -> 2
- net Net-(U7-Pad3): track 0.00 -> 109.8 mm, vias 0 -> 3
- net Net-(U5-Pad10): track 0.00 -> 93.9 mm, vias 0 -> 2
- net /SWR: track 0.00 -> 70.0 mm, vias 0 -> 4
- net /T1: track 0.00 -> 64.0 mm, vias 0 -> 2
- net /SHIFT: track 0.00 -> 57.2 mm, vias 0 -> 2
- net /~{SWR}: track 0.00 -> 56.2 mm, vias 0 -> 2
- net /CTRL_LATCH: track 0.00 -> 55.8 mm, vias 0 -> 1
- net /~{SRD}: track 2.54 -> 50.1 mm, vias 0 -> 1
- net /T9: track 0.00 -> 45.7 mm, vias 0 -> 1
- net /SCLK: track 219.8 -> 262.7 mm, vias 6 -> 8
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Other:
- board text added: "PainfulDiodes BeanBoardSPI"
- board text removed: "PainfulDiodes"

Commit message: Update BeanBoardSPI.kicad_pcb
Parts:
- J1: footprint Connector_PinHeader_2.54mm:PinHeader_1x03_P2.54mm_Vertical -> AltFootprints:PinHeader_1x03_P2.54mm_Vertical
- J12, J13: footprint Connector_PinHeader_2.54mm:PinHeader_1x10_P2.54mm_Vertical -> AltFootprints:PinHeader_1x10_P2.54mm_Vertical
- J2, J3: footprint Connector_PinHeader_2.54mm:PinHeader_1x16_P2.54mm_Vertical -> AltFootprints:PinHeader_1x16_P2.54mm_Vertical
Routing:
- net Net-(U5-Pad13): track 0.00 -> 72.0 mm, vias 0 -> 4
- net Net-(U5-Pad2): track 0.00 -> 51.1 mm, vias 0 -> 2
- net Net-(U5-Pad10): track 93.9 -> 134.6 mm, vias 2 -> 3
- net Net-(JP2-A): track 0.00 -> 32.9 mm, vias 0 -> 1
- net Net-(U6-Pad8): track 0.00 -> 24.5 mm, vias 0 -> 2
- net Net-(U6-Pad4): track 0.00 -> 16.3 mm, vias 0 -> 1
- net Net-(JP3-A): track 0.00 -> 15.5 mm
- net Net-(U9B-D): track 0.00 -> 11.1 mm
- net Net-(U9A-D): track 0.00 -> 11.1 mm
- net Net-(U5-Pad12): track 0.00 -> 11.1 mm
- net /D4: track 71.9 -> 69.2 mm
- net /D5: track 63.1 -> 60.4 mm
- net Net-(U5-Pad3): track 0.00 -> 2.54 mm
Other:
- board text added: "VIN 3V3 GND SCK MISO MOSI CS"

Commit message: Update BeanBoardSPI.kicad_pcb
Routing:
- net /~{WR}: track 64.4 -> 61.7 mm
- net /CLK: track 153.9 -> 151.6 mm
Changed lines of the file:
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@@
     )
     (pad_to_mask_clearance 0)
-    (grid_origin 287.274745 55.810314)
+    (grid_origin 105.156745 -1.085686)
     (pcbplotparams
       (layerselection 0x00010fc_ffffffff)
@@
   (segment (start 179.917087 41.736314) (end 186.878078 41.736314) (width 0.25) (layer "F.Cu") (net 20))
   (via (at 156.464745 42.856314) (size 0.8) (drill 0.4) (layers "F.Cu" "B.Cu") (net 20))
-  (segment (start 189.992745 47.936314) (end 189.987745 47.941314) (width 0.25) (layer "B.Cu") (net 20))
-  (segment (start 188.003078 42.861314) (end 189.992745 42.861314) (width 0.25) (layer "B.Cu") (net 20))
-  (segment (start 189.992745 42.861314) (end 189.992745 47.936314) (width 0.25) (layer "B.Cu") (net 20))
+  (segment (start 188.003078 42.861314) (end 189.484745 44.342981) (width 0.25) (layer "B.Cu") (net 20))
+  (segment (start 189.484745 46.459647) (end 188.003078 47.941314) (width 0.25) (layer "B.Cu") (net 20))
   (segment (start 156.573298 42.747761) (end 156.464745 42.856314) (width 0.25) (layer "B.Cu") (net 20))
   (segment (start 156.573298 19.989406) (end 156.573298 42.747761) (width 0.25) (layer "B.Cu") (net 20))
-  (segment (start 189.987745 47.941314) (end 188.003078 47.941314) (width 0.25) (layer "B.Cu") (net 20))
+  (segment (start 189.484745 44.342981) (end 189.484745 46.459647) (width 0.25) (layer "B.Cu") (net 20))
   (segment (start 161.653298 19.989406) (end 161.689745 20.025853) (width 0.25) (layer "B.Cu") (net 22))
   (segment (start 161.689745 40.461314) (end 162.814745 41.586314) (width 0.25) (layer "B.Cu") (net 22))
@@
   (via (at 270.764745 43.364314) (size 0.8) (drill 0.4) (layers "F.Cu" "B.Cu") (net 24))
   (segment (start 270.510745 18.218314) (end 270.510745 23.298314) (width 0.25) (layer "B.Cu") (net 24))
-  (segment (start 270.510745 23.298314) (end 270.510745 43.110314) (width 0.25) (layer "B.Cu") (net 24))
+  (segment (start 270.764745 43.364314) (end 270.764745 28.124314) (width 0.25) (layer "B.Cu") (net 24))
   (segment (start 270.510745 43.110314) (end 270.764745 43.364314) (width 0.25) (layer "B.Cu") (net 24))
-  (segment (start 270.510745 25.584314) (end 268.224745 25.584314) (width 0.25) (layer "B.Cu") (net 24))
-  (segment (start 270.510745 23.298314) (end 270.510745 25.584314) (width 0.25) (layer "B.Cu") (net 24))
+  (segment (start 270.764745 28.124314) (end 268.224745 25.584314) (width 0.25) (layer "B.Cu") (net 24))
+  (segment (start 270.510745 23.298314) (end 268.224745 25.584314) (width 0.25) (layer "B.Cu") (net 24))
   (segment (start 201.676745 46.666314) (end 201.661745 46.681314) (width 0.25) (layer "F.Cu") (net 27))
   (segment (start 174.353298 30.410314) (end 174.447298 30.316314) (width 0.25) (layer "F.Cu") (net 27))
